File: brd/usb-power-dist.kicad_pcb (KiCad board)
At the start: 2 copper layers, 50 x 50 mm, 38 parts, among them J1 POWER IN, J2 USB_A, J3 USB_A, J4 CASC IN, J5 CASC OUT, U1 TPS2552D, U2 TPS2552D, U3 TPS2513

Commit message: resuelto contorno PCB, verificadas dimensiones, comprobado trazado y colocados componentes restantes -wip
Parts:
- removed the REF** at (190.5, 108.1)
- added REF**: MountingHole_3.2mm_M3_DIN965, Mounting_Holes:MountingHole_3.2mm_M3_DIN965, F.Cu at (149.6, 98.8)
- moved J1 44.8 mm to (144.6, 89.5), turned to 180 degrees
- moved J4 7.29 mm to (132.3, 84.2)
Routing:
- net +5V: track 177.3 -> 205.9 mm
- net GND: track 55.5 -> 32.9 mm
Other:
- outline, holes or cut-outs redrawn
- board text added: "[ ] Comprobar footprints de conectores [X] Ubicación de montaje [X] Verificar forma de placa [X] Trazado completo [ ] Colocar serigrafia [ ] Añadir textos y logos"
- board text removed: "Comprobar footprints de conectores Ubicación de montaje Verificar forma de placa Trazado completo?? Colocar serigrafia Añadir textos y logos"

Commit message: comprobada PCB
Parts:
- added REF**: Symbol_GNU-GPL_CopperTop_Small, Symbols:Symbol_GNU-GPL_CopperTop_Small, B.Cu at (150.6, 90.9)
- added REF***: OSHW-Symbol_8.9x8mm_SilkScreen, Symbols:OSHW-Symbol_8.9x8mm_SilkScreen, B.Cu at (151.6, 100.3)
- moved REF** 2.87 mm to (151.6, 100.8)
Other:
- board text added: "+"
- board text added: "+5V ±5% Only"
- board text added: "-"
- board text added: "Copyright © 2017 kwendenarmo https://github.com/akornsys-rdi/USB-power-dist"
- board text added: "Cover if unused"
- board text added: "Released under GNU/GPL 3 License https://www.gnu.org/licenses/gpl.html"
- board text added: "SPMDBC"
- board text added: "Sch Pcb Mechanical 3D Doc BoM Commercial use"
- board text added: "USB power distribution board"
- board text added: "[X] Comprobar footprints de conectores [X] Ubicación de montaje [X] Verificar forma de placa [X] Trazado completo [X] Colocar serigrafia [X] Añadir textos, polaridad y logos"
- board text removed: "[ ] Comprobar footprints de conectores [X] Ubicación de montaje [X] Verificar forma de placa [X] Trazado completo [ ] Colocar serigrafia [ ] Añadir textos y logos"
