File: brd/usb-power-dist.kicad_pcb (KiCad board)
At the start: 2 copper layers, 50 x 50 mm, 39 parts, among them J1 POWER IN, J2 CASC IN, J3 CASC OUT, J4 USB_A, J5 USB_A, U1 TPS2552D, U2 TPS2552D, U3 TPS2513

Commit message: ordenadas librerias
Parts:
- removed the G*** at (145.5, 100.1)
- added G***: LOGO, lib:akorn-logo-small, F.Cu at (145.5, 100.1)
Changed lines of the file:
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@@
 (kicad_pcb (version 4) (host pcbnew 4.0.7-e2-6376~58~ubuntu16.04.1)
   (general
-    (links 70)
+    (links 0)
     (no_connects 0)
-    (area 101.330001 62.705 205.957143 139.733001)
+    (area 101.330001 62.705 189.174429 139.733001)
     (thickness 1.6)
     (drawings 88)
@@
     )
   )
-  (module brd:akorn-logo-small (layer F.Cu)
+  (module lib:akorn-logo-small (layer F.Cu)
     (at 145.542 100.076)
     (fp_text reference G*** (at 0 0) (layer F.SilkS) hide
